File: PCB_Creation/FeasibilityPCB_production/GPIOExpander/220217_GPIOExpanderAW9523/220217_GPIOExpanderAW9523.kicad_sch (KiCad schematic)
At the start: 53 parts, among them IC1 AW9523BTQR, J1 PWR_Bottom1, J2 PWR_Bottom2, J3 P0_0-07, J4 P0_0-07, J5 I2C ComPort, J6 PWR_Top, J7 Conn_02x08_Odd_Even, J8 Conn_01x08_Male, J9 Conn_01x08_Male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

Commit message: MCU Folder Added
Parts:
- C1: LCSC (none) -> LMK212ABJ106KG8T; Manufacturer_Part_Number (none) -> LMK212ABJ106KG8T
- C2: LCSC (none) -> C0805C104K5RAC7411; Manufacturer_Part_Number (none) -> C0805C104K5RAC7411; PartNumber (none) -> C0805C104K5RAC7411
- D1, D13, D2, D3, D4, D5, D9: LCSC (none) -> APTD2012LZGCK; Manufacturer_Part_Number (none) -> APTD2012LZGCK
- D10: LCSC (none) -> APTD2012LSYCK; Manufacturer_Part_Number (none) -> APTD2012LSYCK
- D11, D7: LCSC (none) -> APTD2012LVBC/D; Manufacturer_Part_Number (none) -> APTD2012LVBC/D
- D12, D8: LCSC (none) -> APTD2012LSURCK; Manufacturer_Part_Number (none) -> APTD2012LSURCK
- D6: value White -> Orange; LCSC (none) -> APT2012LSECK/J4-PRV; Manufacturer_Part_Number (none) -> APT2012LSECK/J4-PRV
- IC1: LCSC (none) -> AW9523BTQR
- J3: footprint Connector_PinHeader_2.54mm:PinHeader_1x07_P2.54mm_Vertical -> Connector_PinHeader_2.54mm:PinHeader_1x08_P2.54mm_Vertical
- J4, J8, J9: LCSC (none) -> M20-9990846; Manufacturer_Part_Number (none) -> M20-9990846
- J7: LCSC (none) -> 5-146265-4; Manufacturer_Part_Number (none) -> 5-146265-4
- R1, R14, R15, R16, R17, R18, R19, R20, R21, R22, R3, R5, R9: LCSC (none) -> ERJ-U06J221V; Manufacturer_Part_Number (none) -> ERJ-U06J221V
- R10, R11, R12, R13, R2, R4, R6, R7, R8: LCSC (none) -> ERJ-6GEYJ103V; Manufacturer_Part_Number (none) -> ERJ-6GEYJ103V
- SW1, SW2, SW3, SW4: LCSC (none) -> 3-1437565-0; Manufacturer_Part_Number (none) -> 3-1437565-0
