File: PCB_Creation/FeasibilityPCB_production/GPIOExpander/220217_GPIOExpanderAW9523/220217_GPIOExpanderAW9523_v02.kicad_sch (KiCad schematic)
At the start: 54 parts, among them IC1 AW9523BTQR, J1 PWR_Bottom1, J2 PWR_Top, J3 PWR_Bottom2, J4 I2C ComPort, J5 P0_0-07, J6 Conn_02x08_Odd_Even, J7 Conn_01x08_Male, J8 Conn_01x08_Male, J9 P0_0-07, SW1 SW_Push, SW2 SW_Push, SW3 SW_Push, SW4 SW_Push

Commit message: Started with version 2 - not finished yet
Parts:
- removed R2: 10k, Resistor_SMD:R_0805_2012Metric, symbol Device:R
- renumbered D7 to D10, D6 to D11, D5 to D12, D4 to D13, D10 to D4, D11 to D5, D13 to D6, D12 to D7, D9 to D8, D8 to D9, J3 to J2, J5 to J3, J9 to J4, J4 to J5, J2 to J6, J6 to J7, J7 to J8, J8 to J9, R6 to R10, R7 to R11, R4 to R12, R18 to R13, R21 to R14, R23 to R15, R22 to R16, R19 to R17, R17 to R18, R15 to R19, R8 to R2, R14 to R20, R13 to R21, R12 to R22, R9 to R3, R10 to R4, R11 to R5, R3 to R6, R5 to R7, R16 to R8, R20 to R9
Connections:
- net P0_7: now also SW1.2; no longer SW1.3
Other:
- moved on the sheet: J5, R12
